Commit message: Add files via upload

File: ur5/urdf/ur5_robot.urdf.xacro (robot description, xacro)
@@ -13,5 +13,5 @@
   <xacro:include filename="$(find ur5)/robotiq_description/urdf/robotiq_85_gripper.urdf.xacro" />
   <xacro:robotiq_85_gripper prefix="" parent="ee_link" >
-	<origin xyz="0.005 0 0" rpy="0 0 0" /> <!-- x must be greater than 0.004 -->
+	<origin xyz="0.005 0 0" rpy="${1.5708} 0 0" /> <!-- x must be greater than 0.004 -->
   </xacro:robotiq_85_gripper>
   <!-- A ground plane -->
@@ -25,4 +25,17 @@
 	<origin xyz="-0.4 1 -0.1" rpy="${1.5708} 0 0 " />
   </xacro:base_ur5>
+  <!-- camerabase -->
+  <xacro:include filename="$(find ur5)/urdf/camera_mount.urdf" />
+  <xacro:camera_mount parent="ee_link" >
+	<origin xyz="${0} ${-(0.3-0.3+0.06)} 0" rpy="0 ${1.5708*2} 0" />
+<!-- change x{0} value for position -->
+  </xacro:camera_mount>
+  <!-- camera -->
+  <xacro:include filename="$(find ur5)/urdf/camera.xacro" />
+  <xacro:camera parent="ee_link" >
+	<origin
+xyz="${-0.005+0} ${-0.09} ${-0.025}" rpy="${-1.5708} ${-1.5708} 0" />
+<!-- change x{0} value for position -->
+  </xacro:camera>
   <link name="world" />
   <joint name="world_joint" type="fixed">

Commit message: Add files via upload

File: ur5/urdf/ur5_robot.urdf.xacro (robot description, xacro)
@@ -34,6 +34,5 @@
   <xacro:include filename="$(find ur5)/urdf/camera.xacro" />
   <xacro:camera parent="ee_link" >
-	<origin
-xyz="${-0.005+0} ${-0.09} ${-0.025}" rpy="${-1.5708} ${-1.5708} 0" />
+	<origin xyz="${-0.005+0} ${-0.09} ${-0.025}" rpy="${-1.5708} ${-1.5708} 0" />
 <!-- change x{0} value for position -->
   </xacro:camera>

Commit message: Camera at the right position

File: ur5/urdf/ur5_robot.urdf.xacro (robot description, xacro)
@@ -13,5 +13,5 @@
   <xacro:include filename="$(find ur5)/robotiq_description/urdf/robotiq_85_gripper.urdf.xacro" />
   <xacro:robotiq_85_gripper prefix="" parent="ee_link" >
-	<origin xyz="0.005 0 0" rpy="${1.5708} 0 0" /> <!-- x must be greater than 0.004 -->
+	<origin xyz="0 0 0" rpy="${1.5708} 0 0" /> <!-- x must be greater than 0.004 -->
   </xacro:robotiq_85_gripper>
   <!-- A ground plane -->
@@ -28,5 +28,5 @@
   <xacro:include filename="$(find ur5)/urdf/camera_mount.urdf" />
   <xacro:camera_mount parent="ee_link" >
-	<origin xyz="${0} ${-(0.3-0.3+0.06)} 0" rpy="0 ${1.5708*2} 0" />
+	<origin xyz="${0.01} ${-(0.3-0.3+0.05)} 0" rpy="0 ${1.5708*2} 0" />
 <!-- change x{0} value for position -->
   </xacro:camera_mount>
@@ -34,5 +34,5 @@
   <xacro:include filename="$(find ur5)/urdf/camera.xacro" />
   <xacro:camera parent="ee_link" >
-	<origin xyz="${-0.005+0} ${-0.09} ${-0.025}" rpy="${-1.5708} ${-1.5708} 0" />
+	<origin xyz="${-0.005+0.01} ${-0.08} ${-0.025}" rpy="${-1.5708} ${-1.5708} 0" />
 <!-- change x{0} value for position -->
   </xacro:camera>

Commit message: Add files via upload

File: ur5/urdf/ur5_robot.urdf.xacro (robot description, xacro)
@@ -13,5 +13,5 @@
   <xacro:include filename="$(find ur5)/robotiq_description/urdf/robotiq_85_gripper.urdf.xacro" />
   <xacro:robotiq_85_gripper prefix="" parent="ee_link" >
-	<origin xyz="0.005 0 0" rpy="0 0 0" /> <!-- x must be greater than 0.004 -->
+	<origin xyz="0 0 0" rpy="${1.5708} 0 0" /> <!-- x must be greater than 0.004 -->
   </xacro:robotiq_85_gripper>
   <!-- A ground plane -->
@@ -25,4 +25,16 @@
 	<origin xyz="-0.4 1 -0.1" rpy="${1.5708} 0 0 " />
   </xacro:base_ur5>
+  <!-- camerabase -->
+  <xacro:include filename="$(find ur5)/urdf/camera_mount.urdf" />
+  <xacro:camera_mount parent="ee_link" >
+	<origin xyz="${0.01} ${-(0.3-0.3+0.05)} 0" rpy="0 ${1.5708*2} 0" />
+<!-- change x{0} value for position -->
+  </xacro:camera_mount>
+  <!-- camera -->
+  <xacro:include filename="$(find ur5)/urdf/camera.xacro" />
+  <xacro:camera parent="ee_link" >
+	<origin xyz="${-0.005+0.01} ${-0.08} ${-0.025}" rpy="${-1.5708} ${-1.5708} 0" />
+<!-- change x{0} value for position -->
+  </xacro:camera>
   <link name="world" />
   <joint name="world_joint" type="fixed">
